Commit message: [3-6] (box) Pick-and-Place 작업 환경 구축 및 그리퍼/박스 모델 반영
- 조작용 박스(Box) 물체 및 3-Table(로봇, 소스, 목적지) 레이아웃 추가
    | MuJoCo 시뮬레이션 내 박스 배치
- 안정적인 파지를 위한 박스 및 그리퍼 패드 물리 속성 강화
    | friction="2.0", condim="6" 및 solimp/solref 접촉 파라미터 최적화
- Robotiq 2F-85 그리퍼 모델링 및 URDF 통합
    | 그리퍼 링크 및 조인트 정의, STL 메시 파일 포함

File: icir_gen3__description/6dof/urdf/GEN3-6DOF_VISION_URDF_ARM_V01.urdf (robot description, URDF)
Before this commit: robot GEN3-6DOF_VISION_URDF_ARM_V01, 9 links, 8 joints
Links:
- added link left_inner_finger, mass 0.0104003125914103; collision mesh filename=package://kortex_description/grippers/robotiq_2f_85/meshes/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 scale=0.001 0.001 0.001; visual mesh filename=package://kortex_description/grippers/robotiq_2f_85/meshes/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 scale=0.001 0.001 0.001
- added link left_inner_finger_pad; collision box size=0.022 0.00635 0.0375; visual box size=0.022 0.00635 0.0375
- added link left_inner_knuckle, mass 0.0271177346495152; collision mesh filename=package://kortex_description/grippers/robotiq_2f_85/meshes/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 scale=0.001 0.001 0.001; visual mesh filename=package://kortex_description/grippers/robotiq_2f_85/meshes/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 scale=0.001 0.001 0.001
- added link left_outer_finger, mass 0.022614240507152; collision mesh filename=package://kortex_description/grippers/robotiq_2f_85/meshes/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 scale=0.001 0.001 0.001; visual mesh filename=package://kortex_description/grippers/robotiq_2f_85/meshes/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 scale=0.001 0.001 0.001
- added link left_outer_knuckle, mass 0.00853198276973456; collision mesh filename=package://kortex_description/grippers/robotiq_2f_85/meshes/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 scale=0.001 0.001 0.001; visual mesh filename=package://kortex_description/grippers/robotiq_2f_85/meshes/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 scale=0.001 0.001 0.001
- added link right_inner_finger, mass 0.0104003125914103; collision mesh filename=package://kortex_description/grippers/robotiq_2f_85/meshes/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 scale=0.001 0.001 0.001; visual mesh filename=package://kortex_description/grippers/robotiq_2f_85/meshes/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 scale=0.001 0.001 0.001
- added link right_inner_finger_pad; collision box size=0.022 0.00635 0.0375; visual box size=0.022 0.00635 0.0375
- added link right_inner_knuckle, mass 0.0271177346495152; collision mesh filename=package://kortex_description/grippers/robotiq_2f_85/meshes/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 scale=0.001 0.001 0.001; visual mesh filename=package://kortex_description/grippers/robotiq_2f_85/meshes/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 scale=0.001 0.001 0.001
- added link right_outer_finger, mass 0.022614240507152; collision mesh filename=package://kortex_description/grippers/robotiq_2f_85/meshes/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 scale=0.001 0.001 0.001; visual mesh filename=package://kortex_description/grippers/robotiq_2f_85/meshes/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 scale=0.001 0.001 0.001
- added link right_outer_knuckle, mass 0.00853198276973456; collision mesh filename=package://kortex_description/grippers/robotiq_2f_85/meshes/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 scale=0.001 0.001 0.001; visual mesh filename=package://kortex_description/grippers/robotiq_2f_85/meshes/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 scale=0.001 0.001 0.001
- added link robotiq_arg2f_base_link, mass 0.22652; collision mesh filename=package://kortex_description/grippers/robotiq_2f_85/meshes/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; visual mesh filename=package://kortex_description/grippers/robotiq_2f_85/meshes/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
Joints:
- added joint finger_joint: type revolute, parent robotiq_arg2f_base_link, child left_outer_knuckle, origin xyz=0 -0.0306011 0.054904 rpy=0 0 3.141592653589793, axis 1 0 0, limit lower=0 upper=0.8 effort=1000 velocity=2.0
- added joint gripper_base_joint: type fixed, parent EndEffector_Link, child robotiq_arg2f_base_link, origin xyz=0.0 0.0 0.0 rpy=0.0 0.0 1.57
- added joint left_inner_finger_joint: type fixed, parent left_outer_finger, child left_inner_finger, origin xyz=0 0.0061 0.0471 rpy=0 0 0, axis 1 0 0, limit lower=-0.8757 upper=0.8757 effort=1000 velocity=2.0, mimic joint=finger_joint multiplier=-1 offset=0
- added joint left_inner_finger_pad_joint: type fixed, parent left_inner_finger, child left_inner_finger_pad, origin xyz=0 -0.0220203446692936 0.03242 rpy=0 0 0, axis 0 0 1
- added joint left_inner_knuckle_joint: type fixed, parent robotiq_arg2f_base_link, child left_inner_knuckle, origin xyz=0 -0.0127 0.06142 rpy=0 0 3.141592653589793, axis 1 0 0, limit lower=0 upper=0.8757 effort=1000 velocity=2.0, mimic joint=finger_joint multiplier=1 offset=0
- added joint left_outer_finger_joint: type fixed, parent left_outer_knuckle, child left_outer_finger, origin xyz=0 0.0315 -0.0041 rpy=0 0 0, axis 1 0 0
- added joint right_inner_finger_joint: type fixed, parent right_outer_finger, child right_inner_finger, origin xyz=0 0.0061 0.0471 rpy=0 0 0, axis 1 0 0, limit lower=-0.8757 upper=0.8757 effort=1000 velocity=2.0, mimic joint=finger_joint multiplier=-1 offset=0
- added joint right_inner_finger_pad_joint: type fixed, parent right_inner_finger, child right_inner_finger_pad, origin xyz=0 -0.0220203446692936 0.03242 rpy=0 0 0, axis 0 0 1
- added joint right_inner_knuckle_joint: type fixed, parent robotiq_arg2f_base_link, child right_inner_knuckle, origin xyz=0 0.0127 0.06142 rpy=0 0 0.0, axis 1 0 0, limit lower=0 upper=0.8757 effort=1000 velocity=2.0, mimic joint=finger_joint multiplier=1 offset=0
- added joint right_outer_finger_joint: type fixed, parent right_outer_knuckle, child right_outer_finger, origin xyz=0 0.0315 -0.0041 rpy=0 0 0, axis 1 0 0
- added joint right_outer_knuckle_joint: type fixed, parent robotiq_arg2f_base_link, child right_outer_knuckle, origin xyz=0 0.0306011 0.054904 rpy=0 0 0, axis 1 0 0, limit lower=0 upper=0.81 effort=1000 velocity=2.0, mimic joint=finger_joint multiplier=1 offset=0
