Commit message: [3-7] (Vision) SAM 기반 Pick-and-Place를 ㄹㅇ뤼한 손목 카메라 및 시뮬레이션 설정 추가
- GEN3-6DOF-VISION_URDF_ARM_V01.xml: Bracelet_Link에 wrist cam 카메라 정의 추가
- kinova_arm_6dof.xml: 오프스크린 렌더링 버퍼(640x480) 설정 추가

File: icir_gen3__description/6dof/urdf/gen3_with_gripper.urdf (robot description, URDF)
Before this commit: robot gen3_robotiq_2f_85_d435, 25 links, 25 joints
Joints:
- joint left_inner_finger_joint: type revolute -> fixed
- joint left_inner_knuckle_joint: type revolute -> fixed
